Commit message: +perception +gripper _control

File: air_description/urdf/air.urdf (robot description, URDF)
Before this commit: robot urdf, 46 links, 45 joints
Links:
- added link root_link
Joints:
- added joint virtual_root_joint: type fixed, parent root_link, child qbhand_base_link, origin xyz=0 0 0  rpy=0 0 0
- joint qbhand_thumb_knuckle_joint: mimic joint=qbhand_synergy_joint multiplier=2.542 -> joint=qbhand_synergy_joint multiplier=1
- joint virtual_camera_joint: origin xyz=0 0 1.3 rpy=0 0.5 0 -> xyz=0 0 1.2 rpy=0 0.5 0
- joint yawj: child qbhand_base_link -> root_link

File: air_moveit_config/config/gazebo_urdf.urdf (robot description, URDF)
Before this commit: robot urdf, 46 links, 45 joints
Links:
- added link root_link
Joints:
- added joint virtual_root_joint: type fixed, parent root_link, child qbhand_base_link, origin xyz=0 0 0  rpy=0 0 0
- joint end_effector_frame_fixed_joint: origin xyz=0 0.275 0 rpy=0 0 0 -> xyz=0 0 0.12 rpy=0 0 0
- joint yawj: child qbhand_base_link -> root_link

Commit message: air_dual_arm urdf added

File: air_description/urdf/air.urdf (robot description, URDF)
Before this commit: robot urdf, 47 links, 46 joints
Joints:
- joint ej: limit lower=-1.4 upper=0.184 effort=0 velocity=0.13 -> lower=-1.4 upper=0.14 effort=0 velocity=0.13
- joint virtual_camera_joint: origin xyz=0 0 1.2 rpy=0 0.5 0 -> xyz=-0.0138 0.0548 1.0685 rpy=0 0.45 -0.1605
